File: hw/interconnects.kicad_sch (KiCad schematic)
At the start: 45 parts, among them J10 SM02B-SRSS-TB, J11 Conn_01x03_MountingPin, J12 Conn_01x03_MountingPin, J13 Conn_01x06_MountingPin, J6 Conn_01x07_MountingPin, J7 Conn_01x08_MountingPin, J8 Conn_01x05_MountingPin, J9 Conn_01x03_MountingPin

Commit message: began with lcsc and footprints
Parts:
- renumbered C41 to C43, C42 to C44, C40 to C45, C36 to C46, C37 to C47, C38 to C48, C39 to C49, C49 to C50, C50 to C51, C47 to C52, C48 to C53, C43 to C54, C44 to C55, C45 to C56, C46 to C57, C60 to C58, C51 to C59, D11 to D10, D14 to D11, D13 to D12, D12 to D13, J9 to J10, J10 to J11, J11 to J4, J7 to J5, J12 to J6, J8 to J7, J6 to J8, J13 to J9, R33 to R27, R27 to R28, R28 to R29, R34 to R30, R38 to R31, R37 to R32, R29 to R33, R30 to R34, R31 to R35, R32 to R36, R36 to R37

Commit message: cleaned up *.kicad_sch
Parts:
- removed C43, C44: C_Small, Capacitor_SMD:C_0603_1608Metric, symbol Device:C_Small
- added C46, C47: 100n X7R 50V, Capacitor_SMD:C_0603_1608Metric, symbol Device:C_Small
- renumbered C45 to C48, C46 to C49, C47 to C50, C48 to C51, C49 to C52, C50 to C53, C51 to C54, C52 to C55, C53 to C56, C54 to C57, C55 to C58, C56 to C59, C57 to C60, C58 to C61, C59 to C62, R24 to R18, R25 to R19, R26 to R20, R27 to R21, R28 to R22, R29 to R23, R30 to R24, R31 to R25, R32 to R26, R33 to R27, R34 to R28, R35 to R29, R36 to R30, R37 to R31
Connections:
- net +3V3: now also C47.1
- net +5V: now also C46.1
- net GND: now also C46.2
Other:
- note added: "[13] Interface - Interconnects."
- moved on the sheet: C48, C49, C50, C51, C52, C53, C54, C55, C56, C57, C58, C59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
