File: hw/interconnects.kicad_sch (KiCad schematic)
At the start: 45 parts, among them J10 Conn_01x03_MountingPin, J11 SM02B-SRSS-TB, J4 Conn_01x03_MountingPin, J5 Conn_01x08_MountingPin, J6 Conn_01x03_MountingPin, J7 Conn_01x05_MountingPin, J8 Conn_01x07_MountingPin, J9 Conn_01x06_MountingPin

Commit message: extended lcsc number coverage and added status led
Parts:
- removed JP1, JP2: SolderJumper_2_Open, Package_SON:WSON-8-1EP_6x5mm_P1.27mm_EP3.4x4mm, symbol Jumper:SolderJumper_2_Open
- removed R18, R19, R20, R23, R28, R29, R30: 100R, Resistor_SMD:R_0201_0603Metric, symbol Device:R_Small
- added JP6: SolderJumper_3_Open, symbol symbols:SolderJumper_3_Open
- D11, D12: value BAT48ZFILM -> B5819W SL; LCSC (none) -> C8598; VFD (none) -> Y
- R21, R24: value 60R4 -> 120 1%; LCSC (none) -> C22787; VFD (none) -> Y
- R22, R27: value 100R -> 120 1%; footprint Resistor_SMD:R_0201_0603Metric -> Resistor_SMD:R_0603_1608Metric; LCSC (none) -> C22787; VFD (none) -> Y
- R25: value 2k -> 2k 1%; footprint Resistor_SMD:R_0201_0603Metric -> Resistor_SMD:R_0402_1005Metric; LCSC (none) -> C4109; VFD (none) -> Y
- R26: value 1k -> 2k 1%; footprint Resistor_SMD:R_0201_0603Metric -> Resistor_SMD:R_0402_1005Metric; LCSC (none) -> C4109; VFD (none) -> Y
- R31: value 10k -> 10k 1%; footprint Resistor_SMD:R_0201_0603Metric -> Resistor_SMD:R_0402_1005Metric; LCSC (none) -> C25744; VFD (none) -> Y
Connections:
- net AUX1: now also J5.3 (Pin_3)
- net AUX2: now also J5.4 (Pin_4)
- net AUX3: now also J5.5 (Pin_5)
- net AUX4: now also J5.6 (Pin_6); no longer R22.2
- net AUX5: now also J5.7 (Pin_7)
- net AUX6: now also J8.3 (Pin_3); no longer R27.2
- net AUX7: now also J8.4 (Pin_4)
- net AUX8: now also J8.5 (Pin_5)
- net AUX9: now also J8.6 (Pin_6)
- net FDCAN_H: now also R21.1, R22.1
- net FDCAN_L: now also R24.2, R27.2
- net at R27.1: now also JP6.1 (A); no longer J8.3 (Pin_3)
- net at C53.1, R24.1: now also R22.2, JP6.2 (C); no longer R21.2
- new net: JP6.3 (B), R21.2
Other:
- moved on the sheet: C53, R21, R24
