File: hw/mcu-power.kicad_sch (KiCad schematic)
At the start: 13 parts, among them U2 STM32G473RCTx

Commit message: basic *.kicad_sch done
Changed lines of the file:
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@@
 (kicad_sch
-	(version 20260826)
+	(version 20260830)
 	(generator "eeschema")
 	(generator_version "10.99")
@@
 	(wire
 		(pts
-			(xy 151.13 62.23) (xy 151.13 64.77)
+			(xy 151.13 63.5) (xy 151.13 64.77)
 		)
 		(stroke
@@
 	(symbol
 		(lib_id "power:+3V3")
-		(at 151.13 62.23 0)
+		(at 151.13 63.5 0)
 		(unit 1)
 		(body_style 1)
@@
 		(in_pos_files yes)
 		(dnp no)
-		(fields_autoplaced yes)
 		(property "Reference" "#PWR04"
-			(at 151.13 66.04 0)
+			(at 151.13 67.31 0)
 			(hide yes)
 			(show_name no)
@@
 		)
 		(property "Value" "+3V3"
-			(at 151.13 57.15 0)
+			(at 151.13 59.182 0)
 			(show_name no)
 			(do_not_autoplace no)
@@
 		)
 		(property "Footprint" ""
-			(at 151.13 62.23 0)
+			(at 151.13 63.5 0)
 			(hide yes)
 			(show_name no)
@@
 		)
 		(property "Datasheet" ""
-			(at 151.13 62.23 0)
+			(at 151.13 63.5 0)
 			(hide yes)
 			(show_name no)
@@
 		)
 		(property "Description" "Power symbol creates a global label with name \"+3V3\""
-			(at 151.13 62.23 0)
-			(hide yes)
-			(show_name no)
+			(at 151.13 63.5 0)
+			(hide yes)
+			(show_name no)

Commit message: began with lcsc and footprints
Parts:
- removed C1, C11, C2, C3, C4, C8: 100n X7R 50V, symbol Device:C
- removed C5: 4u7 X7R 16V, symbol Device:C
- removed C6: 100n X7R 10V, symbol Device:C
- added C1, C11, C3, C4, C5, C6, C8: 100n X7R 50V, Capacitor_SMD:C_0603_1608Metric, symbol Device:C_Small
- added C62: 4u7 X5R 16V, Capacitor_SMD:C_0603_1608Metric, symbol Device:C
- C10: value 4u7 X7R 10V -> 4u7 X5R 16V; footprint (none) -> Capacitor_SMD:C_0603_1608Metric; LCSC (none) -> C19666
- C7, C9: value 1u X7R 10V -> 1u X5R 50V; footprint (none) -> Capacitor_SMD:C_0603_1608Metric; LCSC (none) -> C15849
- FB1: footprint (none) -> Inductor_SMD:L_0603_1608Metric; LCSC (none) -> C14709
- renumbered U2 to U1
Connections:
- net +3V3: now also C1.1, C3.1, C4.1, C5.1, C6.1, C62.1
- net +3V3A: now also C11.1, C8.1
- net GND: now also C1.2, C11.2, C3.2, C4.2, C5.2, C6.2, C62.2, C8.2
Other:
- moved on the sheet: FB1

Commit message: cleaned up *.kicad_sch
Parts:
- renumbered C62 to C2
Connections:
- net +3V3: no longer C9.1, FB1.1
- net +3V3A: now also C9.1, FB1.1; no longer C10.1, C11.1, C7.1, C8.1, FB1.2, U1.28 (VREF+), U1.29 (VDDA)
- new net: C10.1, C11.1, C7.1, C8.1, FB1.2, U1.28 (VREF+), U1.29 (VDDA)
Other:
- note added: "MCU Power Supply"
- note added: "[4] MCU - Power"
- title: (none) -> MCU - Power
- moved on the sheet: C1, C10, C11, C2, C3, C4, C5, C6, C7, C8, C9, FB1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
