File: hw/mcu-power.kicad_sch (KiCad schematic)
At the start: 13 parts, among them U1 STM32G473RCTx

Commit message: extended lcsc number coverage and added status led
Parts:
- FB1: VFD (none) -> Y
Changed lines of the file:
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@@
 			)
 		)
-		(property "VFD" ""
+		(property "VFD" "Y"
 			(at 130.81 111.76 90)
 			(hide yes)
