File: hw/sense_pos.kicad_sch (KiCad schematic)
At the start: 2 parts, among them U4 AS5047D

Commit message: began with lcsc and footprints
Parts:
- removed C61: 4u7 X7R 10V, symbol Device:C
- added C42: 4u7 X5R 16V, Capacitor_SMD:C_0603_1608Metric, symbol Device:C
Connections:
- net +3V3: now also C42.1
- net GND: now also C42.2
Changed lines of the file:
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@@
 		(dnp no)
 		(fields_autoplaced yes)
-		(property "Reference" "#PWR027"
+		(property "Reference" "#PWR044"
 			(at 152.4 121.92 0)
 			(hide yes)
@@
 			(project "atlas-electronics"
 				(path "/915bc1ff-7be5-4368-a2db-c4889af73afd/b136d1dc-418d-4dd5-9857-4058e82b2897"
-					(reference "#PWR027")
+					(reference "#PWR044")
 					(unit 1)
 				)
@@
 		(in_pos_files yes)
 		(dnp no)
-		(property "Reference" "#PWR080"
+		(property "Reference" "#PWR043"
 			(at 170.18 107.95 0)
 			(hide yes)
@@
 			(project "atlas-electronics"
 				(path "/915bc1ff-7be5-4368-a2db-c4889af73afd/b136d1dc-418d-4dd5-9857-4058e82b2897"
-					(reference "#PWR080")
+					(reference "#PWR043")
 					(unit 1)
 				)
@@
 		(in_pos_files yes)
 		(dnp no)
-		(property "Reference" "C61"
+		(property "Reference" "C42"
 			(at 172.974 109.22 0)
 			(show_name no)
@@
 			)
 		)
-		(property "Value" "4u7 X7R 10V"
+		(property "Value" "4u7 X5R 16V"
 			(at 172.974 111.76 0)
 			(show_name no)
@@
 			)
 		)
-		(property "Footprint" ""
+		(property "Footprint" "Capacitor_SMD:C_0603_1608Metric"
 			(at 171.1452 114.3 0)
 			(hide yes)
@@
 			)
 		)
+		(property "LCSC" "C19666"
+			(at 170.18 110.49 0)
+			(hide yes)
+			(show_name no)
+			(do_not_autoplace no)
+			(effects
+				(font
+					(size 1.016 1.016)
+				)
+			)
+		)
 		(pin "2"
 		)
@@
 			(project "atlas-electronics"
 				(path "/915bc1ff-7be5-4368-a2db-c4889af73afd/b136d1dc-418d-4dd5-9857-4058e82b2897"
-					(reference "C61")
+					(reference "C42")
 					(unit 1)
 				)
@@
 		(dnp no)
 		(fields_autoplaced yes)
-		(property "Reference" "#PWR026"
+		(property "Reference" "#PWR042"
 			(at 152.4 88.9 0)
 			(hide yes)
@@
 			(project "atlas-electronics"
 				(path "/915bc1ff-7be5-4368-a2db-c4889af73afd/b136d1dc-418d-4dd5-9857-4058e82b2897"
-					(reference "#PWR026")
+					(reference "#PWR042")
 					(unit 1)
 				)
@@
 		(dnp no)
 		(fields_autoplaced yes)
-		(property "Reference" "#PWR081"
+		(property "Reference" "#PWR045"
 			(at 170.18 121.92 0)
 			(hide yes)
@@
 			(project "atlas-electronics"
 				(path "/915bc1ff-7be5-4368-a2db-c4889af73afd/b136d1dc-418d-4dd5-9857-4058e82b2897"
-					(reference "#PWR081")
-					(unit 1)
-				)
+					(reference "#PWR045")
+					(unit 1)
+				)

Commit message: cleaned up *.kicad_sch
Parts:
- renumbered C42 to C39, U4 to U3
Other:
- note added: "Position Sensing"
- note added: "[10] Sensing - Position"
- moved on the sheet: C39, U3
