File: hw/sense_vbat.kicad_sch (KiCad schematic)
At the start: 5 parts

Commit message: began with lcsc and footprints
Parts:
- removed C34, C35: 100n, symbol Device:C
- removed R22, R23: 10k, LED_SMD:LED_SK6805_PLCC4_2.4x2.7mm_P1.3mm, symbol Device:R
- added C40, C41: 100n X7R 50V, Capacitor_SMD:C_0603_1608Metric, symbol Device:C_Small
- added R13, R17: 10k 1%, Resistor_SMD:R_0603_1608Metric, symbol Device:R
- TH1: footprint Resistor_SMD:R_0805_2012Metric -> Resistor_SMD:R_0603_1608Metric; LCSC (none) -> C13564
Connections:
- net +3V3: now also R13.1, R17.1
- net GND: now also C40.2, C41.2
- net NTC_INVERTER: now also C40.1, R13.2
- net NTC_MOTOR: now also C41.1, R17.2

Commit message: cleaned up *.kicad_sch
Parts:
- renumbered C40 to C37, C41 to C38, R13 to R16
Other:
- note added: "Temperature Sensing"
- note added: "[9] Sensing - Temperature"
- moved on the sheet: C37, C38, R16, R17, TH1
