File: hw/sense_vbat.kicad_sch (KiCad schematic)
At the start: 5 parts

Commit message: extended lcsc number coverage and added status led
Parts:
- R16, R17: footprint Resistor_SMD:R_0603_1608Metric -> Resistor_SMD:R_0402_1005Metric; LCSC C25804 -> C25744; VFD (none) -> Y
Changed lines of the file:
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@@
 			)
 		)
-		(property "Footprint" "Resistor_SMD:R_0603_1608Metric"
+		(property "Footprint" "Resistor_SMD:R_0402_1005Metric"
 			(at 155.702 78.74 90)
 			(hide yes)
@@
 			)
 		)
-		(property "LCSC" "C25804"
+		(property "LCSC" "C25744"
 			(at 157.48 78.74 0)
 			(hide yes)
@@
 			)
 		)
-		(property "VFD" ""
+		(property "VFD" "Y"
 			(at 157.48 78.74 0)
 			(hide yes)
@@
 			)
 		)
-		(property "Footprint" "Resistor_SMD:R_0603_1608Metric"
+		(property "Footprint" "Resistor_SMD:R_0402_1005Metric"
 			(at 104.902 78.74 90)
 			(hide yes)
@@
 			)
 		)
-		(property "LCSC" "C25804"
+		(property "LCSC" "C25744"
 			(at 106.68 78.74 0)
 			(hide yes)
@@
 			)
 		)
-		(property "VFD" ""
+		(property "VFD" "Y"
 			(at 106.68 78.74 0)
 			(hide yes)
