File: hw/Power.kicad_sch (KiCad schematic)
At the start: 22 parts, among them U6 AP2112K-3.3, U7 TPS7A20xxxDBV

Commit message: extended lcsc number coverage and added status led
Parts:
- C65, C66, C67, C68: value 1u C0G 50V -> 1u 7XR 25V
- D1: value SS16 -> SS14; footprint Diode_SMD:D_SOD-123 -> Diode_SMD:D_SMA; LCSC C18199176 -> C2480; VFD (none) -> Y
- D14, D15, R2: VFD (none) -> Y
- L1: LCSC C341059 -> (none)
- R3: value 54k9 -> 54k9 1%; footprint (none) -> Resistor_SMD:R_0603_1608Metric; LCSC (none) -> C23206; VFD (none) -> Y
- R4: value 10k -> 10k 1%; footprint (none) -> Resistor_SMD:R_0402_1005Metric; LCSC (none) -> C25744; VFD (none) -> Y
Changed lines of the file:
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@@
 			)
 		)
-		(property "LCSC" "C341059"
+		(property "LCSC" ""
 			(at 172.72 67.31 90)
 			(hide yes)
@@
 			)
 		)
-		(property "Value" "SS16"
+		(property "Value" "SS14"
 			(at 163.83 72.0724 90)
 			(show_name no)
@@
 			)
 		)
-		(property "Footprint" "Diode_SMD:D_SOD-123"
+		(property "Footprint" "Diode_SMD:D_SMA"
 			(at 161.29 71.12 0)
 			(hide yes)
@@
 			)
 		)
-		(property "LCSC" "C18199176"
+		(property "LCSC" "C2480"
 			(at 161.29 71.12 90)
 			(hide yes)
@@
 			)
 		)
-		(property "VFD" ""
+		(property "VFD" "Y"
 			(at 161.29 71.12 90)
 			(hide yes)
@@
 			)
 		)
-		(property "VFD" ""
+		(property "VFD" "Y"
 			(at 204.47 129.54 90)
 			(hide yes)
@@
 			)
 		)
-		(property "Value" "10k"
+		(property "Value" "10k 1%"
 			(at 181.61 85.0899 0)
 			(show_name no)
@@
 			)
 		)
-		(property "Footprint" ""
+		(property "Footprint" "Resistor_SMD:R_0402_1005Metric"
 			(at 177.292 83.82 90)
 			(hide yes)
@@
 			)
 		)
-		(property "VFD" ""
+		(property "VFD" "Y"
+			(at 179.07 83.82 0)
+			(hide yes)
+			(show_name no)
+			(do_not_autoplace no)
+			(effects
+				(font
+					(size 1.016 1.016)
+				)
+			)
+		)
+		(property "LCSC" "C25744"
 			(at 179.07 83.82 0)
 			(hide yes)
@@
 			)
 		)
-		(property "Value" "1u C0G 50V"
+		(property "Value" "1u 7XR 25V"
 			(at 178.054 130.81 0)
 			(show_name no)
@@
 			)
 		)
-		(property "VFD" ""
+		(property "VFD" "Y"
 			(at 195.58 129.54 90)
 			(hide yes)
@@
 			)
 		)
-		(property "Value" "1u C0G 50V"
+		(property "Value" "1u 7XR 25V"
 			(at 122.174 129.54 0)
 			(show_name no)
@@
 			)
 		)
-		(property "Value" "1u C0G 50V"
+		(property "Value" "1u 7XR 25V"
 			(at 142.748 130.81 0)
 			(show_name no)
@@
 			)
 		)
-		(property "VFD" ""
+		(property "VFD" "Y"
 			(at 116.84 67.31 90)
 			(hide yes)
@@
 			)
 		)
-		(property "Value" "1u C0G 50V"
+		(property "Value" "1u 7XR 25V"
 			(at 86.868 129.54 0)
 			(show_name no)
@@
 			)
 		)
-		(property "Value" "54k9"
+		(property "Value" "54k9 1%"
 			(at 181.61 74.9299 0)
 			(show_name no)
@@
 			)
 		)
-		(property "Footprint" ""
+		(property "Footprint" "Resistor_SMD:R_0603_1608Metric"
 			(at 177.292 73.66 90)
 			(hide yes)
@@
 			)
 		)
-		(property "VFD" ""
+		(property "VFD" "Y"
+			(at 179.07 73.66 0)
+			(hide yes)
+			(show_name no)
+			(do_not_autoplace no)
+			(effects
+				(font
+					(size 1.016 1.016)
+				)
+			)
+		)
+		(property "LCSC" "C23206"
 			(at 179.07 73.66 0)
 			(hide yes)
