File: hw/gate-driver.kicad_sch (KiCad schematic)
At the start: 8 parts

Commit message: extended lcsc number coverage and added status led
Parts:
- R1: footprint Resistor_SMD:R_0603_1608Metric -> Resistor_SMD:R_0402_1005Metric; LCSC C25804 -> C25744; VFD (none) -> Y
Changed lines of the file:
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@@
 			)
 		)
-		(property "Footprint" "Resistor_SMD:R_0603_1608Metric"
+		(property "Footprint" "Resistor_SMD:R_0402_1005Metric"
 			(at 115.062 80.01 90)
 			(hide yes)
@@
 			)
 		)
-		(property "LCSC" "C25804"
+		(property "LCSC" "C25744"
 			(at 116.84 80.01 0)
 			(hide yes)
@@
 			)
 		)
-		(property "VFD" ""
+		(property "VFD" "Y"
 			(at 116.84 80.01 0)
 			(hide yes)
