File: hw/mcu.kicad_sch (KiCad schematic)
At the start: 30 parts, among them U1 STM32G473RCTx

Commit message: extended lcsc number coverage and added status led
Connections:
- net STATUS_LED_SIMPLE: now reaches U1.26 (PB2)
- no-connect marks 5 -> 4
Changed lines of the file:
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@@
 	)
 	(no_connect
-		(at 73.66 92.71)
-	)
-	(no_connect
 		(at 43.18 125.73)
 	)
@@
 	(wire
 		(pts
+			(xy 73.66 92.71) (xy 96.52 92.71)
+		)
+		(stroke
+			(width 0)
+			(type default)
+		)
+	)
+	(wire
+		(pts
 			(xy 110.49 113.03) (xy 129.54 113.03)
 		)
@@
 	(wire
 		(pts
+			(xy 186.69 107.95) (xy 220.98 107.95)
+		)
+		(stroke
+			(width 0)
+			(type default)
+		)
+	)
+	(wire
+		(pts
 			(xy 246.38 134.62) (xy 265.43 134.62)
 		)
@@
 		)
 	)
+	(label "STATUS_LED_SIMPLE"
+		(at 96.52 92.71 180)
+		(effects
+			(font
+				(size 1.27 1.27)
+			)
+			(justify right bottom)
+		)
+	)
 	(label "FDCAN_RX"
 		(at 110.49 113.03 0)
@@
 		)
 	)
+	(label "STATUS_LED_SIMPLE"
+		(at 186.69 107.95 0)
+		(effects
+			(font
+				(size 1.27 1.27)
+			)
+			(justify left bottom)
+		)
+	)
 	(label "NTC_INVERTER"
 		(at 110.49 166.37 0)
@@
 		(effects
 			(font
+				(size 1.27 1.27)
+			)
+			(justify left)
+		)
+	)
+	(hierarchical_label "STATUS_LED_SIMPLE"
+		(shape output)
+		(at 220.98 107.95 0)
+		(effects
+			(font
