File: hw/misc.kicad_sch (KiCad schematic)
At the start: 14 parts, among them Y1 Crystal_GND24

Commit message: extended lcsc number coverage and added status led
Parts:
- C63, C64: value 10pF X7R 50V -> 10pF C0G 50V; VFD (none) -> Y
- R32, R33, R34: value 10k -> 10k 1%; footprint (none) -> Resistor_SMD:R_0402_1005Metric; LCSC (none) -> C25744; VFD (none) -> Y
- Y1: VFD (none) -> Y
Changed lines of the file:
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@@
 			)
 		)
-		(property "Value" "10k"
+		(property "Value" "10k 1%"
 			(at 74.93 85.0899 0)
 			(show_name no)
@@
 			)
 		)
-		(property "Footprint" ""
+		(property "Footprint" "Resistor_SMD:R_0402_1005Metric"
 			(at 70.612 83.82 90)
 			(hide yes)
@@
 			)
 		)
-		(property "VFD" ""
+		(property "VFD" "Y"
+			(at 72.39 83.82 0)
+			(hide yes)
+			(show_name no)
+			(do_not_autoplace no)
+			(effects
+				(font
+					(size 1.016 1.016)
+				)
+			)
+		)
+		(property "LCSC" "C25744"
 			(at 72.39 83.82 0)
 			(hide yes)
@@
 			)
 		)
-		(property "Value" "10k"
+		(property "Value" "10k 1%"
 			(at 66.04 85.0899 0)
 			(show_name no)
@@
 			)
 		)
-		(property "Footprint" ""
+		(property "Footprint" "Resistor_SMD:R_0402_1005Metric"
 			(at 61.722 83.82 90)
 			(hide yes)
@@
 			)
 		)
-		(property "VFD" ""
+		(property "VFD" "Y"
+			(at 63.5 83.82 0)
+			(hide yes)
+			(show_name no)
+			(do_not_autoplace no)
+			(effects
+				(font
+					(size 1.016 1.016)
+				)
+			)
+		)
+		(property "LCSC" "C25744"
 			(at 63.5 83.82 0)
 			(hide yes)
@@
 			)
 		)
-		(property "VFD" ""
+		(property "VFD" "Y"
 			(at 196.85 105.41 0)
 			(hide yes)
@@
 			)
 		)
-		(property "Value" "10k"
+		(property "Value" "10k 1%"
 			(at 57.15 85.0899 0)
 			(show_name no)
@@
 			)
 		)
-		(property "Footprint" ""
+		(property "Footprint" "Resistor_SMD:R_0402_1005Metric"
 			(at 56.388 83.82 90)
 			(hide yes)
@@
 			)
 		)
-		(property "VFD" ""
+		(property "VFD" "Y"
+			(at 54.61 83.82 0)
+			(hide yes)
+			(show_name no)
+			(do_not_autoplace no)
+			(effects
+				(font
+					(size 1.016 1.016)
+				)
+			)
+		)
+		(property "LCSC" "C25744"
 			(at 54.61 83.82 0)
 			(hide yes)
@@
 			)
 		)
-		(property "Value" "10pF X7R 50V"
+		(property "Value" "10pF C0G 50V"
 			(at 180.34 111.76 0)
 			(show_name no)
@@
 			)
 		)
-		(property "VFD" ""
+		(property "VFD" "Y"
 			(at 187.96 110.49 0)
 			(hide yes)
@@
 			)
 		)
-		(property "Value" "10pF X7R 50V"
+		(property "Value" "10pF C0G 50V"
 			(at 208.28 111.7599 0)
 			(show_name no)
@@
 			)
 		)
-		(property "VFD" ""
+		(property "VFD" "Y"
 			(at 205.74 110.49 0)
 			(hide yes)
