File: hw/status-led.kicad_sch (KiCad schematic)
At the start: 12 parts, among them U3 SN74LV1T125DCK

Commit message: began with lcsc and footprints
Parts:
- removed C52, C53, C54, C55, C56, C57: C_Small, Capacitor_SMD:C_0603_1608Metric, symbol Device:C_Small
- added C33, C34, C35, C36, C37, C38: 100n X7R 50V, Capacitor_SMD:C_0603_1608Metric, symbol Device:C_Small
- D5, D6, D7, D8, D9: LCSC (none) -> C2909056
- U3: LCSC (none) -> C75925
Connections:
- net +5V: now also C33.1, C34.1, C35.1, C36.1, C37.1, C38.1
- net GND: now also C33.2, C34.2, C35.2, C36.2, C37.2, C38.2
Other:
- note added: "Either SK6805 ec15 is small or sk6805 micro j bigger"

Commit message: cleaned up *.kicad_sch
Parts:
- D5, D6, D7, D8, D9: footprint LED_SMD:LED_SK6805_PLCC4_2.4x2.7mm_P1.3mm -> LED_SMD:LED_SK6812_EC15_1.5x1.5mm; LCSC C2909056 -> C2890035
- renumbered C33 to C40, C34 to C41, C35 to C42, C36 to C43, C37 to C44, C38 to C45, U3 to U4
Other:
- note added: "Status LEDs"
- note added: "[11] Interface - Status LEDs"
- title: (none) -> Status LED
- moved on the sheet: C40, C41, C42, C43, C44, C45, D5, U4

Commit message: extended lcsc number coverage
Parts:
- C40, C41, C42, C43, C44, C45: footprint Capacitor_SMD:C_0603_1608Metric -> Capacitor_SMD:C_0402_1005Metric; LCSC C14663 -> C307331; VFD (none) -> Y
Changed lines of the file:
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@@
 			)
 		)
-		(property "Footprint" "Capacitor_SMD:C_0603_1608Metric"
+		(property "Footprint" "Capacitor_SMD:C_0402_1005Metric"
 			(at 125.73 82.55 0)
 			(hide yes)
@@
 			)
 		)
-		(property "LCSC" "C14663"
+		(property "LCSC" "C307331"
 			(at 125.73 82.55 0)
 			(hide yes)
@@
 				(font
 					(size 1.27 1.27)
+				)
+			)
+		)
+		(property "VFD" "Y"
+			(at 125.73 82.55 0)
+			(hide yes)
+			(show_name no)
+			(do_not_autoplace no)
+			(effects
+				(font
+					(size 1.016 1.016)
 				)
 			)
@@
 			)
 		)
+		(property "VFD" ""
+			(at 121.92 97.79 0)
+			(hide yes)
+			(show_name no)
+			(do_not_autoplace no)
+			(effects
+				(font
+					(size 1.016 1.016)
+				)
+			)
+		)
 		(pin "2"
 		)
@@
 			)
 		)
-		(property "Footprint" "Capacitor_SMD:C_0603_1608Metric"
+		(property "Footprint" "Capacitor_SMD:C_0402_1005Metric"
 			(at 95.25 82.55 0)
 			(hide yes)
@@
 			)
 		)
-		(property "LCSC" "C14663"
+		(property "LCSC" "C307331"
 			(at 95.25 82.55 0)
 			(hide yes)
@@
 				(font
 					(size 1.27 1.27)
+				)
+			)
+		)
+		(property "VFD" "Y"
+			(at 95.25 82.55 0)
+			(hide yes)
+			(show_name no)
+			(do_not_autoplace no)
+			(effects
+				(font
+					(size 1.016 1.016)
 				)
 			)
@@
 			)
 		)
-		(property "Footprint" "Capacitor_SMD:C_0603_1608Metric"
+		(property "Footprint" "Capacitor_SMD:C_0402_1005Metric"
 			(at 168.91 82.55 0)
 			(hide yes)
@@
 			)
 		)
-		(property "LCSC" "C14663"
+		(property "LCSC" "C307331"
 			(at 168.91 82.55 0)
 			(hide yes)
@@
 				(font
 					(size 1.27 1.27)
+				)
+			)
+		)
+		(property "VFD" "Y"
+			(at 168.91 82.55 0)
+			(hide yes)
+			(show_name no)
+			(do_not_autoplace no)
+			(effects
+				(font
+					(size 1.016 1.016)
 				)
 			)
@@
 			)
 		)
-		(property "Footprint" "Capacitor_SMD:C_0603_1608Metric"
+		(property "Footprint" "Capacitor_SMD:C_0402_1005Metric"
 			(at 190.5 82.55 0)
 			(hide yes)
@@
 			)
 		)
-		(property "LCSC" "C14663"
+		(property "LCSC" "C307331"
 			(at 190.5 82.55 0)
 			(hide yes)
@@
 				(font
 					(size 1.27 1.27)
+				)
+			)
+		)
+		(property "VFD" "Y"
+			(at 190.5 82.55 0)
+			(hide yes)
+			(show_name no)
+			(do_not_autoplace no)
+			(effects
+				(font
+					(size 1.016 1.016)
 				)
 			)
@@
 			)
 		)
+		(property "VFD" ""
+			(at 143.51 97.79 0)
+			(hide yes)
+			(show_name no)
+			(do_not_autoplace no)
+			(effects
+				(font
+					(size 1.016 1.016)
+				)
+			)
+		)
 		(pin "2"
 		)
@@
 			)
 		)
+		(property "VFD" ""
+			(at 91.44 97.79 0)
+			(hide yes)
+			(show_name no)
+			(do_not_autoplace no)
+			(effects
+				(font
+					(size 1.016 1.016)
+				)
+			)
+		)
 		(pin "2"
 		)
@@
 			)
 		)
+		(property "VFD" ""
+			(at 165.1 97.79 0)
+			(hide yes)
+			(show_name no)
+			(do_not_autoplace no)
+			(effects
+				(font
+					(size 1.016 1.016)
+				)
+			)
+		)
 		(pin "2"
 		)
@@
 			)
 		)
-		(property "Footprint" "Capacitor_SMD:C_0603_1608Metric"
+		(property "Footprint" "Capacitor_SMD:C_0402_1005Metric"
 			(at 147.32 82.55 0)
 			(hide yes)
@@
 			)
 		)
-		(property "LCSC" "C14663"
+		(property "LCSC" "C307331"
 			(at 147.32 82.55 0)
 			(hide yes)
@@
 				(font
 					(size 1.27 1.27)
+				)
+			)
+		)
+		(property "VFD" "Y"
+			(at 147.32 82.55 0)
+			(hide yes)
+			(show_name no)
+			(do_not_autoplace no)
+			(effects
+				(font
+					(size 1.016 1.016)
 				)
 			)
@@
 			)
 		)
-		(property "Footprint" "Capacitor_SMD:C_0603_1608Metric"
+		(property "Footprint" "Capacitor_SMD:C_0402_1005Metric"
 			(at 212.09 82.55 0)
 			(hide yes)
@@
 			)
 		)
-		(property "LCSC" "C14663"
+		(property "LCSC" "C307331"
 			(at 212.09 82.55 0)
 			(hide yes)
@@
 				(font
 					(size 1.27 1.27)
+				)
+			)
+		)
+		(property "VFD" "Y"
+			(at 212.09 82.55 0)
+			(hide yes)
+			(show_name no)
+			(do_not_autoplace no)
+			(effects
+				(font
+					(size 1.016 1.016)
 				)
 			)
@@
 			)
 		)
+		(property "VFD" ""
+			(at 186.69 97.79 0)
+			(hide yes)
+			(show_name no)
+			(do_not_autoplace no)
+			(effects
+				(font
+					(size 1.016 1.016)
+				)
+			)
+		)
 		(pin "2"
 		)
@@
 				)
 			)
+		)
+		(property "VFD" ""
+			(at 208.28 97.79 0)
+			(hide yes)
+			(show_name no)
+			(do_not_autoplace no)
+			(effects
+				(font
+					(size 1.016 1.016)
+				)
+			)

Commit message: extended lcsc number coverage and added status led
Parts:
- D5, D6, D7, D8, D9: LCSC C2890035 -> (none)
- U4: LCSC C75925 -> (none)
Changed lines of the file:
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@@
+	(wire
+		(pts
+			(xy 80.01 127) (xy 81.28 127)
+		)
+		(stroke
+			(width 0)
+			(type default)
+		)
+	)
 	(wire
 		(pts
@@
 			(width 0)
 			(type default)
+		)
+	)
+	(hierarchical_label "STATUS_LED_SIMPLE"
+		(shape input)
+		(at 81.28 127 180)
+		(effects
+			(font
+				(size 1.016 1.016)
+			)
+			(justify right)
 		)
 	)
@@
 			)
 		)
-		(property "LCSC" "C2890035"
+		(property "LCSC" ""
 			(at 121.92 97.79 0)
 			(hide yes)
@@
 			)
 		)
-		(property "LCSC" "C2890035"
+		(property "LCSC" ""
 			(at 143.51 97.79 0)
 			(hide yes)
@@
 			)
 		)
-		(property "LCSC" "C75925"
+		(property "LCSC" ""
 			(at 91.44 97.79 0)
 			(hide yes)
@@
 			)
 		)
-		(property "LCSC" "C2890035"
+		(property "LCSC" ""
 			(at 165.1 97.79 0)
 			(hide yes)
@@
 			)
 		)
-		(property "LCSC" "C2890035"
+		(property "LCSC" ""
 			(at 186.69 97.79 0)
 			(hide yes)
@@
 			)
 		)
-		(property "LCSC" "C2890035"
+		(property "LCSC" ""
 			(at 208.28 97.79 0)
 			(hide yes)
