File: hw/inverter.kicad_sch (KiCad schematic)
At the start: 22 parts, among them J1 Conn_01x01, Q1 ISC025N06LM6, Q4 ISC025N06LM6

Commit message: extended lcsc number coverage and added status led
Parts:
- D2: value 1A 40V -> B5819W SL; VFD (none) -> Y
Changed lines of the file:
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@@
 			)
 		)
-		(property "Value" "1A 40V"
+		(property "Value" "B5819W SL"
 			(at 24.13 157.1624 90)
 			(show_name no)
@@
 			)
 		)
-		(property "VFD" ""
+		(property "VFD" "Y"
 			(at 21.59 156.21 90)
 			(hide yes)

Commit message: reviewed by pz
Parts:
- removed C23: 220u 20% 35V, Capacitor_SMD:CP_Elec_8x10.5, symbol Device:C_Polarized
- removed D2: B5819W SL, Diode_SMD:D_SOD-123, symbol Device:D_Schottky
- removed TP15, TP16, TP17, TP18, TP19, TP20, TP21, TP22, TP23: TestPoint, TestPoint:TestPoint_Pad_D1.0mm, symbol Connector:TestPoint
- added C23, C34, C73, C74: 3n3 X7R 100V, Capacitor_SMD:C_0603_1608Metric, symbol Device:C
- added C26, C27, C28, C29, C31, C32, C35, C70, C71, C76, C77, C78, C79, C80: 10u X5R 50V, Capacitor_SMD:C_1206_3216Metric, symbol Device:C
- added C30, C75: 100n X7R 50V, Capacitor_SMD:C_0402_1005Metric, symbol Device:C_Small
- added C72, C81: 220u 20% 35V, Capacitor_SMD:CP_Elec_8x10.5, symbol Device:C_Polarized
- added J2, J3: Conn_01x01, A_pad:Goated holy pad, symbol Connector_Generic:Conn_01x01
- added Q2, Q3, Q5, Q6: ISC025N06LM6, Package_TO_SOT_SMD:TDSON-8-1, symbol Transistor_FET:CSD18532Q5B
- added R10, R6, R7, R9: 5R, symbol Device:R
- added R12, R13: 2m 3W 1%, Resistor_SMD:R_2512_6332Metric, symbol Device:R
- added R47, R48, R49, R50, R51, R52: 0R, Resistor_SMD:R_0603_1608Metric_Pad0.98x0.95mm_HandSolder, symbol Device:R
- C22: now fitted
- C25: value 4u7 X7R 50V -> 10u X5R 50V; LCSC C29823 -> C13585
Connections:
- net +VBAT: now also C26.1, C27.1, C28.1, C29.1, C30.1, C31.1, C32.1, C35.1, C70.1, C71.1, C72.1, C75.1, C76.1, C77.1, C78.1, C79.1, C80.1, C81.1, Q2.5 (D), Q3.5 (D), R6.2, R7.2
- net GHA: now also R48.1, R49.1, R51.1; no longer Q1.4 (G)
- net GLA: now also R47.1, R50.1, R52.1; no longer Q4.4 (G)
- net GND: now also C24.2, C26.2, C27.2, C28.2, C29.2, C30.2, C31.2, C32.2, C35.2, C70.2, C71.2, C72.2, C75.2, C76.2, C77.2, C78.2, C79.2, C80.2, C81.2, R12.2, R13.2
- net SHA: now also C23.2, C34.1, C73.2, C74.1, J2.1 (Pin_1), J3.1 (Pin_1), Q2.1 (S), Q2.2 (S), Q2.3 (S), Q3.1 (S), Q3.2 (S), Q3.3 (S), Q5.5 (D), Q6.5 (D)
- net SNUBH_A: now also C23.1, C73.1, R6.1, R7.1
- net SNUBL_A: now also C34.2, C74.2, R10.2, R9.2
- net SPA: now also Q5.1 (S), Q5.2 (S), Q5.3 (S), Q6.1 (S), Q6.2 (S), Q6.3 (S), R10.1, R12.1, R13.1, R9.1; no longer C24.2
- new net: Q5.4 (G), R50.2
- new net: Q6.4 (G), R52.2
- new net: Q2.4 (G), R49.2
- new net: Q1.4 (G), R48.2
- new net: Q3.4 (G), R51.2
- new net: Q4.4 (G), R47.2
Other:
- moved on the sheet: C24, C25

Commit message: improved schem
Parts:
- R10, R5, R6, R7, R8, R9: footprint (none) -> Resistor_SMD:R_0603_1608Metric_Pad0.98x0.95mm_HandSolder
Changed lines of the file:
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@@
 			)
 		)
-		(property "Footprint" ""
+		(property "Footprint" "Resistor_SMD:R_0603_1608Metric_Pad0.98x0.95mm_HandSolder"
 			(at 70.358 138.43 90)
 			(hide yes)
@@
 			)
 		)
-		(property "Footprint" ""
+		(property "Footprint" "Resistor_SMD:R_0603_1608Metric_Pad0.98x0.95mm_HandSolder"
 			(at 191.008 138.43 90)
 			(hide yes)
@@
 			)
 		)
-		(property "Footprint" ""
+		(property "Footprint" "Resistor_SMD:R_0603_1608Metric_Pad0.98x0.95mm_HandSolder"
 			(at 311.658 102.87 90)
 			(hide yes)
@@
 			)
 		)
-		(property "Footprint" ""
+		(property "Footprint" "Resistor_SMD:R_0603_1608Metric_Pad0.98x0.95mm_HandSolder"
 			(at 311.658 138.43 90)
 			(hide yes)
@@
 			)
 		)
-		(property "Footprint" ""
+		(property "Footprint" "Resistor_SMD:R_0603_1608Metric_Pad0.98x0.95mm_HandSolder"
 			(at 191.008 102.87 90)
 			(hide yes)
@@
 			)
 		)
-		(property "Footprint" ""
+		(property "Footprint" "Resistor_SMD:R_0603_1608Metric_Pad0.98x0.95mm_HandSolder"
 			(at 70.358 102.87 90)
 			(hide yes)
