File: hw/_restore_backup_2026-09-28T13-11-11-751/Power.kicad_sch (KiCad schematic)
At the start: 22 parts, among them U6 AP2112K-3.3, U7 TPS7A20xxxDBV

Commit message: extended lcsc number coverage
Parts:
- C18: footprint Capacitor_SMD:C_0402_1005Metric -> Capacitor_SMD:C_0603_1608Metric; LCSC C307331 -> C14663; VFD Y -> (none)
- C19: VFD Y -> (none)
- C20: footprint Capacitor_SMD:C_0603_1608Metric -> Capacitor_SMD:C_0805_2012Metric; LCSC C96446 -> C15850; VFD Y -> (none)
- C65, C66, C67, C68: value 1u C0G 50V -> 1u X7R 25V; footprint Capacitor_SMD:C_0402_1005Metric -> Capacitor_SMD:C_0603_1608Metric; VFD Y -> (none)
