File: hw/_restore_backup_2026-09-28T13-11-11-751/interconnects.kicad_sch (KiCad schematic)
At the start: 45 parts, among them J10 Conn_01x03_MountingPin, J11 SM02B-SRSS-TB, J4 Conn_01x03_MountingPin, J5 Conn_01x08_MountingPin, J6 Conn_01x03_MountingPin, J7 Conn_01x05_MountingPin, J8 Conn_01x07_MountingPin, J9 Conn_01x06_MountingPin

Commit message: extended lcsc number coverage
Parts:
- C46, C47: footprint Capacitor_SMD:C_0402_1005Metric -> Capacitor_SMD:C_0603_1608Metric; LCSC C307331 -> C14663; VFD Y -> (none)
- C53: value 4.7nF X7R 50V -> C_Small; footprint Capacitor_SMD:C_0402_1005Metric -> Capacitor_SMD:C_0603_1608Metric; LCSC C1538 -> (none); VFD Y -> (none)
- C54, C61: value 100n X7R 50V -> 100n; footprint Capacitor_SMD:C_0402_1005Metric -> Package_DFN_QFN:WDFN-10-1EP_3x3mm_P0.5mm_EP1.8x2.5mm; LCSC C307331 -> (none); VFD Y -> (none)
- C55, C56: value 100n X7R 50V -> C_Small; footprint Capacitor_SMD:C_0402_1005Metric -> Capacitor_SMD:C_0603_1608Metric; LCSC C307331 -> (none); VFD Y -> (none)
- C62: value 100n X7R 50V -> C_Small; footprint Capacitor_SMD:C_0402_1005Metric -> Package_DFN_QFN:WDFN-10-1EP_3x3mm_P0.5mm_EP1.8x2.5mm; LCSC C307331 -> (none); VFD Y -> (none)
Connections:
- net GND: now also C56.2
