File: hw/_restore_backup_2026-09-28T13-11-11-751/inverter.kicad_sch (KiCad schematic)
At the start: 22 parts, among them J1 Conn_01x01, Q1 ISC025N06LM6, Q4 ISC025N06LM6

Commit message: extended lcsc number coverage
Parts:
- C24: footprint Capacitor_SMD:C_0402_1005Metric -> Capacitor_SMD:C_0603_1608Metric; LCSC C307331 -> C14663; VFD Y -> (none)
- C25: VFD Y -> (none)
