File: hw/_restore_backup_2026-09-28T13-11-11-751/misc.kicad_sch (KiCad schematic)
At the start: 14 parts, among them Y1 Crystal_GND24

Commit message: extended lcsc number coverage
Parts:
- C63, C64: value 10pF X7R 50V -> 10pF; footprint Capacitor_SMD:C_0402_1005Metric -> Capacitor_SMD:C_0603_1608Metric; LCSC C32949 -> (none)
Changed lines of the file:
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@@
-			)
-		)
-		(property "VFD" ""
-			(at 72.39 83.82 0)
-			(hide yes)
-			(show_name no)
-			(do_not_autoplace no)
-			(effects
-				(font
-					(size 1.016 1.016)
-				)
 			)
 		)
@@
 			)
 		)
-		(property "VFD" ""
-			(at 63.5 102.87 90)
-			(hide yes)
-			(show_name no)
-			(do_not_autoplace no)
-			(effects
-				(font
-					(size 1.016 1.016)
-				)
-			)
-		)
 		(pin "2"
 		)
@@
 			)
 		)
-		(property "VFD" ""
-			(at 54.61 173.99 0)
-			(hide yes)
-			(show_name no)
-			(do_not_autoplace no)
-			(effects
-				(font
-					(size 1.016 1.016)
-				)
-			)
-		)
 		(pin "1"
 		)
@@
 			)
 		)
-		(property "VFD" ""
-			(at 72.39 102.87 90)
-			(hide yes)
-			(show_name no)
-			(do_not_autoplace no)
-			(effects
-				(font
-					(size 1.016 1.016)
-				)
-			)
-		)
 		(pin "2"
 		)
@@
 			)
 		)
-		(property "VFD" ""
-			(at 77.47 173.99 0)
-			(hide yes)
-			(show_name no)
-			(do_not_autoplace no)
-			(effects
-				(font
-					(size 1.016 1.016)
-				)
-			)
-		)
 		(pin "1"
 		)
@@
 			)
 		)
-		(property "VFD" ""
-			(at 204.47 88.9 90)
-			(hide yes)
-			(show_name no)
-			(do_not_autoplace no)
-			(effects
-				(font
-					(size 1.016 1.016)
-				)
-			)
-		)
 		(pin "2"
 		)
@@
 			)
 		)
-		(property "VFD" ""
-			(at 54.61 102.87 90)
-			(hide yes)
-			(show_name no)
-			(do_not_autoplace no)
-			(effects
-				(font
-					(size 1.016 1.016)
-				)
-			)
-		)
 		(pin "2"
 		)
@@
 			)
 		)
-		(property "VFD" ""
-			(at 123.19 173.99 0)
-			(hide yes)
-			(show_name no)
-			(do_not_autoplace no)
-			(effects
-				(font
-					(size 1.016 1.016)
-				)
-			)
-		)
 		(pin "1"
 		)
@@
 			)
 		)
-		(property "VFD" ""
-			(at 63.5 83.82 0)
-			(hide yes)
-			(show_name no)
-			(do_not_autoplace no)
-			(effects
-				(font
-					(size 1.016 1.016)
-				)
-			)
-		)
 		(pin "2"
 		)
@@
 			)
 		)
-		(property "VFD" ""
-			(at 196.85 105.41 0)
-			(hide yes)
-			(show_name no)
-			(do_not_autoplace no)
-			(effects
-				(font
-					(size 1.016 1.016)
-				)
-			)
-		)
 		(pin "4"
 		)
@@
 			)
 		)
-		(property "VFD" ""
-			(at 100.33 173.99 0)
-			(hide yes)
-			(show_name no)
-			(do_not_autoplace no)
-			(effects
-				(font
-					(size 1.016 1.016)
-				)
-			)
-		)
 		(pin "1"
 		)
@@
 			)
 		)
-		(property "VFD" ""
-			(at 54.61 83.82 0)
-			(hide yes)
-			(show_name no)
-			(do_not_autoplace no)
-			(effects
-				(font
-					(size 1.016 1.016)
-				)
-			)
-		)
 		(pin "2"
 		)
@@
 			)
 		)
-		(property "Value" "10pF X7R 50V"
+		(property "Value" "10pF"
 			(at 180.34 111.76 0)
 			(show_name no)
@@
 			)
 		)
-		(property "Footprint" "Capacitor_SMD:C_0402_1005Metric"
+		(property "Footprint" "Capacitor_SMD:C_0603_1608Metric"
 			(at 187.96 110.49 0)
 			(hide yes)
@@
 			)
 		)
-		(property "VFD" ""
-			(at 187.96 110.49 0)
-			(hide yes)
-			(show_name no)
-			(do_not_autoplace no)
-			(effects
-				(font
-					(size 1.016 1.016)
-				)
-			)
-		)
-		(property "LCSC" "C32949"
-			(at 187.96 110.49 0)
-			(hide yes)
-			(show_name no)
-			(do_not_autoplace no)
-			(effects
-				(font
-					(size 1.016 1.016)
-				)
-			)
-		)
 		(pin "1"
 		)
@@
 			)
 		)
-		(property "Value" "10pF X7R 50V"
+		(property "Value" "10pF"
 			(at 208.28 111.7599 0)
 			(show_name no)
@@
 			)
 		)
-		(property "Footprint" "Capacitor_SMD:C_0402_1005Metric"
+		(property "Footprint" "Capacitor_SMD:C_0603_1608Metric"
 			(at 205.74 110.49 0)
 			(hide yes)
@@
 				)
 			)
-		)
-		(property "VFD" ""
-			(at 205.74 110.49 0)
-			(hide yes)
-			(show_name no)
-			(do_not_autoplace no)
-			(effects
-				(font
-					(size 1.016 1.016)
-				)
-			)
-		)
-		(property "LCSC" "C32949"
-			(at 205.74 110.49 0)
-			(hide yes)
-			(show_name no)
-			(do_not_autoplace no)
-			(effects
-				(font
-					(size 1.016 1.016)
-				)
-			)
