File: hw/_restore_backup_2026-09-28T13-11-11-751/sense_pos.kicad_sch (KiCad schematic)
At the start: 2 parts, among them U3 AS5047D

Commit message: extended lcsc number coverage
Parts:
- C39: VFD Y -> (none)
Changed lines of the file:
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@@
-			)
-		)
-		(property "VFD" "Y"
-			(at 137.16 109.22 0)
-			(hide yes)
-			(show_name no)
-			(do_not_autoplace no)
-			(effects
-				(font
-					(size 1.016 1.016)
-				)
 			)
 		)
@@
 				)
 			)
-		)
-		(property "VFD" ""
-			(at 119.38 99.06 0)
-			(hide yes)
-			(show_name no)
-			(do_not_autoplace no)
-			(effects
-				(font
-					(size 1.016 1.016)
-				)
-			)
