File: hw/_restore_backup_2026-09-28T13-11-11-751/sense_temp.kicad_sch (KiCad schematic)
At the start: 2 parts, among them U5 TCAN334G

Commit message: extended lcsc number coverage
Parts:
- removed C69: 100n X7R 50V, Capacitor_SMD:C_0402_1005Metric, symbol Device:C_Small
- removed U5: TCAN334G, Package_SO:TSSOP-14_4.4x5mm_P0.65mm, symbol Interface_CAN_LIN:TCAN334G
- added C36: 10n X7R 50V, Capacitor_SMD:C_0603_1608Metric, symbol Device:C_Small
- added R14: 100k 1%, Resistor_SMD:R_0603_1608Metric, symbol Device:R
- added R15: 10k 1%, Resistor_SMD:R_0603_1608Metric, symbol Device:R
Connections:
- net GND: now also C36.2, R15.2
- new net +VBAT: R14.1
- new net SENSE_VBAT: C36.1, R14.2, R15.1
- no-connect marks 2 -> 0
Other:
- note added: "VBAT Sensing"
- note added: "[8] Sensing - VBAT"
- note removed: "FDCAN Transceiver"
- note removed: "[12] Interface - FDCAN Tran."
