File: hw/_restore_backup_2026-09-28T13-11-11-751/status-led.kicad_sch (KiCad schematic)
At the start: 14 parts, among them Y1 Crystal_GND24

Commit message: extended lcsc number coverage
Parts:
- removed C63, C64: 10pF X7R 50V, Capacitor_SMD:C_0402_1005Metric, symbol Device:C_Small
- removed H1, H2, H3, H4: MountingHole_Pad, symbol Mechanical:MountingHole_Pad
- removed JP3, JP4, JP5: SolderJumper_2_Open, Package_SON:WSON-8-1EP_6x5mm_P1.27mm_EP3.4x4mm, symbol Jumper:SolderJumper_2_Open
- removed R32, R33, R34: 10k, symbol Device:R
- removed R35: 0R, symbol Device:R
- removed Y1: Crystal_GND24, Crystal:Crystal_SMD_3225-4Pin_3.2x2.5mm, symbol Device:Crystal_GND24
- added C40, C41, C42, C43, C44, C45: 100n X7R 50V, Capacitor_SMD:C_0603_1608Metric, symbol Device:C_Small
- added D5, D6, D7, D8, D9: SK6805, LED_SMD:LED_SK6812_EC15_1.5x1.5mm, symbol LED:SK6805
- added U4: SN74LV1T125DCK, Package_TO_SOT_SMD:SOT-353_SC-70-5, symbol Logic_LevelTranslator:SN74LV1T125DCK
Connections:
- net GND: now also C40.2, C41.2, C42.2, C43.2, C44.2, C45.2, D5.2 (VSS), D6.2 (VSS), D7.2 (VSS), D8.2 (VSS), D9.2 (VSS), U4.1 (~{OE}), U4.3 (GND)
- new net: D5.1 (DOUT), D6.3 (DIN)
- new net: D5.3 (DIN), U4.4 (Y)
- new net: D6.1 (DOUT), D7.3 (DIN)
- new net: D7.1 (DOUT), D8.3 (DIN)
- new net: D8.1 (DOUT), D9.3 (DIN)
- new net +5V: C40.1, C41.1, C42.1, C43.1, C44.1, C45.1, D5.4 (VDD), D6.4 (VDD), D7.4 (VDD), D8.4 (VDD), D9.4 (VDD), U4.5 (VCC)
- new net STATUS_LED: U4.2 (A)
- no-connect marks 0 -> 1
Other:
- note added: "Either SK6805 ec15 is small or sk6805 micro j bigger"
- note added: "Status LEDs"
- note added: "[11] Interface - Status LEDs"
- note removed: "Crystal"
- note removed: "Mounting Holes"
- note removed: "UID"
- note removed: "[13] MISC."
- title: (none) -> Status LED
