File: hw/_restore_backup_2026-10-01T07-45-20-214/interconnects.kicad_sch (KiCad schematic)
At the start: 46 parts, among them J10 Conn_01x03_MountingPin, J11 SM02B-SRSS-TB, J4 Conn_01x03_MountingPin, J5 Conn_01x08_MountingPin, J6 Conn_01x03_MountingPin, J7 Conn_01x05_MountingPin, J8 Conn_01x07_MountingPin, J9 Conn_01x06_MountingPin

Commit message: reviewed by pz
Connections:
- net at JP6.1 (A), R27.1: no longer R24.1
- net at C53.1, JP6.2 (C): now also R22.2, R24.1
- net at JP6.3 (B), R21.2: no longer R22.2
Other:
- note added: "AUX 1"
- note added: "AUX 2"
- note added: "EXT Homing Hall"
- note removed: "AUX1"
- note removed: "AUX2"
- note removed: "CAN"
- note removed: "Ext. Homing Interrupt"
- note removed: "SPI"
- moved on the sheet: C54, J7
