File: hw/_restore_backup_2026-10-01T07-45-20-214/status-led.kicad_sch (KiCad schematic)
At the start: 12 parts, among them U4 SN74LV1T125DCK

Commit message: reviewed by pz
Changed lines of the file:
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@@
+	(wire
+		(pts
+			(xy 80.01 127) (xy 81.28 127)
+		)
+		(stroke
+			(width 0)
+			(type default)
+		)
+	)
 	(wire
 		(pts
@@
 		)
 	)
+	(hierarchical_label "STATUS_LED_SIMPLE"
+		(shape input)
+		(at 81.28 127 180)
+		(effects
+			(font
+				(size 1.016 1.016)
+			)
+			(justify right)
+		)
+	)
